File: broads/rp2040/i2s_audio_recorder/i2s_audio_recorder.kicad_sch (KiCad schematic)
At the start: 55 parts, among them J1 USB_C_Receptacle_USB2.0_16P, J2 Conn_01x04_Pin, J3 SD_Card_Device, J4 Conn_01x08_Pin, J5 Conn_01x08_Pin, J6 Conn_01x08_Pin, U1 MSM261S4030H0R, U1 SMBJ5.0CA, U2 RP2040, U3 SMBJ5.0CA, U4 SMBJ5.0CA, U5 AMS1117-3.3, U7 W25Q128JVS, Y1 12M

Commit message: Update signature of all schematics
Other:
- company: Krysztal Huang -> Krysztal Huang <krysztal.huang@outlook.com>
Changed lines of the file:
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@@
 		(date "2024-09-01")
 		(rev "0.1.0")
-		(company "Krysztal Huang")
+		(company "Krysztal Huang <krysztal.huang@outlook.com>")
 	)
 	(junction
