File: slices/i2s/msm261s4030h0r/msm261s4030h0r.kicad_sch (KiCad schematic)
At the start: 3 parts, among them U1 MSM261S4030H0R

Commit message: Update signature of all schematics
Other:
- company: (none) -> Krysztal Huang <krysztal.huang@outlook.com>
Changed lines of the file:
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@@
 	(generator_version "8.0")
 	(paper "A4")
+	(title_block
+		(date "2024-9-19")
+		(company "Krysztal Huang <krysztal.huang@outlook.com>")
+	)
 	(junction
 		(at 182.88 85.09)
